File: dcdc_7909.sch (KiCad schematic (older format))
At the start: 28 parts, among them J1 V_IN, J2 G_IN, J3 +10V, J4 G_OUT, J5 -10V, U1 TMR6, U2 LT3045xMSE, U3 LT3094xMSE

Commit message: Update the files.
Parts:
- U1: symbol marcin_library:TMR6 -> dcdc_7909-rescue:TMR6-marcin_library
- U3: symbol Regulator_Linear2:LT3094xMSE -> dcdc_7909-rescue:LT3094xMSE-Regulator_Linear2
Connections:
- wire segments 100 -> 99
- no-connect marks 0 -> 1
Changed lines of the file:
@@
 Comment4 ""
 $EndDescr
-$Comp
-L marcin_library:TMR6 U1
-U 1 1 5E9E1524
-P 2800 3500
-F 0 "U1" H 2800 3625 50  0000 C CNN
-F 1 "TMR6" H 2800 3534 50  0000 C CNN
-F 2 "marcin_library:Traco_TMR6" H 2800 3500 50  0001 C CNN
-F 3 "" H 2800 3500 50  0001 C CNN
-	1    2800 3500
-	1    0    0    -1
-$EndComp
-Wire Wire Line
-	2300 3800 1650 3800
 Wire Wire Line
 	1650 3800 1650 3700
@@
 $EndComp
 $Comp
-L Regulator_Linear2:LT3094xMSE U3
+L dcdc_7909-rescue:LT3094xMSE-Regulator_Linear2 U3
 U 1 1 5E9E8A2D
 P 7150 4450
@@
 	1    0    0    -1
 $EndComp
+$Comp
+L dcdc_7909-rescue:TMR6-marcin_library U1
+U 1 1 5E9E1524
+P 2800 3500
+F 0 "U1" H 2800 3625 50  0000 C CNN
+F 1 "TMR6" H 2800 3534 50  0000 C CNN
+F 2 "marcin_library:Traco_TMR6" H 2800 3500 50  0001 C CNN
+F 3 "" H 2800 3500 50  0001 C CNN
+	1    2800 3500
+	1    0    0    -1
+$EndComp
+NoConn ~ 2300 3800
 $EndSCHEMATC
