File: dcdc_7909.kicad_sch (KiCad schematic)
At the start: 64 parts, among them J1 V_IN, J2 G_IN, J3 +10V, J4 G_OUT, J5 -10V, J6 Conn_01x01, J7 Conn_01x01, J8 Conn_01x01, J9 Conn_01x01, U1 LM2940-SOT223-15, U2 MAXM15068AMB+, U3 MAX17579ATC+, U4 LT3045xMSE, U5 LT3094xMSE

Commit message: Calculated the resistor values.
Parts:
- R3: value 1M07 1% -> 499k 1%
- R4: value 150k 1% -> 47k 1%
- R8: value 1M07 1% -> 19k1 1%
- R9: value 150k 1% -> 1.78 1%
Changed lines of the file:
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@@
       (effects (font (size 1.27 1.27)) (justify left))
     )
-    (property "Value" "1M07 1%" (id 1) (at 135.763 83.312 0)
+    (property "Value" "499k 1%" (id 1) (at 135.763 83.312 0)
       (effects (font (size 1.27 1.27)) (justify left))
     )
@@
       (effects (font (size 1.27 1.27)) (justify left))
     )
-    (property "Value" "150k 1%" (id 1) (at 135.763 92.837 0)
+    (property "Value" "47k 1%" (id 1) (at 135.763 92.837 0)
       (effects (font (size 1.27 1.27)) (justify left))
     )
@@
       (effects (font (size 1.27 1.27)) (justify left))
     )
-    (property "Value" "1M07 1%" (id 1) (at 169.418 138.557 0)
+    (property "Value" "19k1 1%" (id 1) (at 169.418 138.557 0)
       (effects (font (size 1.27 1.27)) (justify left))
     )
@@
       (effects (font (size 1.27 1.27)) (justify left))
     )
-    (property "Value" "150k 1%" (id 1) (at 169.418 149.987 0)
+    (property "Value" "1.78 1%" (id 1) (at 169.418 149.987 0)
       (effects (font (size 1.27 1.27)) (justify left))
     )
@@
     )
     (path "/7f91b756-389f-49ac-b079-1019353cb179"
-      (reference "R3") (unit 1) (value "1M07 1%") (footprint "Resistor_SMD:R_0402_1005Metric")
+      (reference "R3") (unit 1) (value "499k 1%") (footprint "Resistor_SMD:R_0402_1005Metric")
     )
     (path "/a28fa307-48fe-450e-9aca-af74a63d6dd0"
-      (reference "R4") (unit 1) (value "150k 1%") (footprint "Resistor_SMD:R_0402_1005Metric")
+      (reference "R4") (unit 1) (value "47k 1%") (footprint "Resistor_SMD:R_0402_1005Metric")
     )
     (path "/203396a4-c02d-43be-8429-5a421ad8ae82"
@@
     )
     (path "/a77b34e3-d8f7-42df-ba35-51ad80d3e4cd"
-      (reference "R8") (unit 1) (value "1M07 1%") (footprint "Resistor_SMD:R_0402_1005Metric")
+      (reference "R8") (unit 1) (value "19k1 1%") (footprint "Resistor_SMD:R_0402_1005Metric")
     )
     (path "/fb3817a9-a3cd-48d2-be88-fc156170e895"
-      (reference "R9") (unit 1) (value "150k 1%") (footprint "Resistor_SMD:R_0402_1005Metric")
+      (reference "R9") (unit 1) (value "1.78 1%") (footprint "Resistor_SMD:R_0402_1005Metric")
     )
     (path "/00000000-0000-0000-0000-00005ea01249"

Commit message: Filled out LCSC components refs.
Parts:
- C10, C13, C14, C4, C7: LCSC C15195 -> C307331
- C12: LCSC C15195 -> C50254
- C5: LCSC C426653 -> C50254; PN Murata GCM32EC71E226KE36 -> (none)
- R1: LCSC C477187 -> C11490
- R11, R13: LCSC C21190 -> C11702
- R2: LCSC C319870 -> C334752
- R3: LCSC C477187 -> C407728
- R4: LCSC C319870 -> C25792
- R5: LCSC C477187 -> C477691
- R6: LCSC C319870 -> C25786
- R7: LCSC C319870 -> C284661
- R8: LCSC C477187 -> C52036
- R9: value 1.78 1% -> 1k78 1%; LCSC C319870 -> C284379
Changed lines of the file:
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@@
       (effects (font (size 1.27 1.27)) hide)
     )
-    (property "LCSC" "C21190" (id 4) (at 231.775 43.815 0)
+    (property "LCSC" "C11702" (id 4) (at 231.775 43.815 0)
       (effects (font (size 1.27 1.27)) hide)
     )
@@
       (effects (font (size 1.27 1.27)) hide)
     )
-    (property "LCSC" "C21190" (id 4) (at 240.665 92.075 0)
+    (property "LCSC" "C11702" (id 4) (at 240.665 92.075 0)
       (effects (font (size 1.27 1.27)) hide)
     )
@@
       (effects (font (size 1.27 1.27)) hide)
     )
-    (property "LCSC" "C15195" (id 4) (at 33.655 74.295 0)
+    (property "LCSC" "C307331" (id 4) (at 33.655 74.295 0)
       (effects (font (size 1.27 1.27)) hide)
     )
@@
       (effects (font (size 1.27 1.27)) hide)
     )
-    (property "LCSC" "C319870" (id 4) (at 42.545 87.63 0)
+    (property "LCSC" "C334752" (id 4) (at 42.545 87.63 0)
       (effects (font (size 1.27 1.27)) hide)
     )
@@
       (effects (font (size 1.27 1.27)) hide)
     )
-    (property "LCSC" "C15195" (id 4) (at 40.64 128.27 0)
+    (property "LCSC" "C307331" (id 4) (at 40.64 128.27 0)
       (effects (font (size 1.27 1.27)) hide)
     )
@@
       (effects (font (size 1.27 1.27)) hide)
     )
-    (property "LCSC" "C477187" (id 4) (at 49.53 130.81 0)
+    (property "LCSC" "C477691" (id 4) (at 49.53 130.81 0)
       (effects (font (size 1.27 1.27)) hide)
     )
@@
       (effects (font (size 1.27 1.27)) hide)
     )
-    (property "LCSC" "C319870" (id 4) (at 49.53 140.97 0)
+    (property "LCSC" "C25786" (id 4) (at 49.53 140.97 0)
       (effects (font (size 1.27 1.27)) hide)
     )
@@
       (effects (font (size 1.27 1.27)) hide)
     )
-    (property "LCSC" "C426653" (id 4) (at 53.975 83.185 0)
-      (effects (font (size 1.27 1.27)) hide)
-    )
-    (property "PN" "Murata GCM32EC71E226KE36" (id 5) (at 53.975 83.185 0)
+    (property "LCSC" "C50254" (id 4) (at 53.975 83.185 0)
+      (effects (font (size 1.27 1.27)) hide)
+    )
+    (property "PN" "" (id 5) (at 53.975 83.185 0)
       (effects (font (size 1.27 1.27)) hide)
     )
@@
       (effects (font (size 1.27 1.27)) hide)
     )
-    (property "LCSC" "C15195" (id 4) (at 77.47 151.13 0)
+    (property "LCSC" "C50254" (id 4) (at 77.47 151.13 0)
       (effects (font (size 1.27 1.27)) hide)
     )
@@
       (effects (font (size 1.27 1.27)) hide)
     )
-    (property "LCSC" "C477187" (id 4) (at 133.985 84.455 0)
+    (property "LCSC" "C407728" (id 4) (at 133.985 84.455 0)
       (effects (font (size 1.27 1.27)) hide)
     )
@@
       (effects (font (size 1.27 1.27)) hide)
     )
-    (property "LCSC" "C15195" (id 4) (at 146.685 133.35 0)
+    (property "LCSC" "C307331" (id 4) (at 146.685 133.35 0)
       (effects (font (size 1.27 1.27)) hide)
     )
@@
       (effects (font (size 1.27 1.27)) hide)
     )
-    (property "LCSC" "C319870" (id 4) (at 133.985 93.98 0)
+    (property "LCSC" "C25792" (id 4) (at 133.985 93.98 0)
       (effects (font (size 1.27 1.27)) hide)
     )
@@
       (effects (font (size 1.27 1.27)) hide)
     )
-    (property "LCSC" "C477187" (id 4) (at 167.64 139.7 0)
+    (property "LCSC" "C52036" (id 4) (at 167.64 139.7 0)
       (effects (font (size 1.27 1.27)) hide)
     )
@@
       (effects (font (size 1.27 1.27)) hide)
     )
-    (property "LCSC" "C319870" (id 4) (at 87.63 151.13 0)
+    (property "LCSC" "C284661" (id 4) (at 87.63 151.13 0)
       (effects (font (size 1.27 1.27)) hide)
     )
@@
       (effects (font (size 1.27 1.27)) hide)
     )
-    (property "LCSC" "C15195" (id 4) (at 127.635 83.185 0)
+    (property "LCSC" "C307331" (id 4) (at 127.635 83.185 0)
       (effects (font (size 1.27 1.27)) hide)
     )
@@
       (effects (font (size 1.27 1.27)) hide)
     )
-    (property "LCSC" "C15195" (id 4) (at 156.21 144.78 0)
+    (property "LCSC" "C307331" (id 4) (at 156.21 144.78 0)
       (effects (font (size 1.27 1.27)) hide)
     )
@@
       (effects (font (size 1.27 1.27)) hide)
     )
-    (property "LCSC" "C477187" (id 4) (at 42.545 78.74 0)
+    (property "LCSC" "C11490" (id 4) (at 42.545 78.74 0)
       (effects (font (size 1.27 1.27)) hide)
     )
@@
       (effects (font (size 1.27 1.27)) (justify left))
     )
-    (property "Value" "1.78 1%" (id 1) (at 169.418 149.987 0)
+    (property "Value" "1k78 1%" (id 1) (at 169.418 149.987 0)
       (effects (font (size 1.27 1.27)) (justify left))
     )
@@
       (effects (font (size 1.27 1.27)) hide)
     )
-    (property "LCSC" "C319870" (id 4) (at 167.64 151.13 0)
+    (property "LCSC" "C284379" (id 4) (at 167.64 151.13 0)
       (effects (font (size 1.27 1.27)) hide)
     )
@@
     )
     (path "/fb3817a9-a3cd-48d2-be88-fc156170e895"
-      (reference "R9") (unit 1) (value "1.78 1%") (footprint "Resistor_SMD:R_0402_1005Metric")
+      (reference "R9") (unit 1) (value "1k78 1%") (footprint "Resistor_SMD:R_0402_1005Metric")
     )
     (path "/00000000-0000-0000-0000-00005ea01249"

Commit message: Fixed the 2u2 cap footprints.
Parts:
- C12, C5: LCSC C50254 -> C377773
- U2: LCSC (none) -> DO NOT POPULATE
- U3: LCSC (none) -> C5691155
Changed lines of the file:
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@@
       (effects (font (size 1.27 1.27) italic) hide)
+    )
+    (property "LCSC" "DO NOT POPULATE" (id 4) (at 111.76 69.215 0)
+      (effects (font (size 1.27 1.27)) hide)
     )
     (pin "1")
@@
       (effects (font (size 1.27 1.27)) hide)
     )
-    (property "LCSC" "C50254" (id 4) (at 53.975 83.185 0)
+    (property "LCSC" "C377773" (id 4) (at 53.975 83.185 0)
       (effects (font (size 1.27 1.27)) hide)
     )
@@
       (effects (font (size 1.27 1.27)) hide)
     )
-    (property "LCSC" "C50254" (id 4) (at 77.47 151.13 0)
+    (property "LCSC" "C377773" (id 4) (at 77.47 151.13 0)
       (effects (font (size 1.27 1.27)) hide)
     )
@@
       (effects (font (size 1.27 1.27) italic) hide)
     )
-    (pin "1")
+    (property "LCSC" "C5691155" (id 4) (at 83.82 124.46 0)
+      (effects (font (size 1.27 1.27)) hide)
+    )
+    (pin "1")

Commit message: Sent for production.
Parts:
- C12, C5: footprint Capacitor_SMD:C_0805_2012Metric -> Capacitor_SMD:C_1206_3216Metric; LCSC C377773 -> C50254
Changed lines of the file:
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@@
       (effects (font (size 1.27 1.27)) (justify left))
     )
-    (property "Footprint" "Capacitor_SMD:C_0805_2012Metric" (id 2) (at 53.975 83.185 0)
+    (property "Footprint" "Capacitor_SMD:C_1206_3216Metric" (id 2) (at 53.975 83.185 0)
       (effects (font (size 1.27 1.27)) hide)
     )
@@
       (effects (font (size 1.27 1.27)) hide)
     )
-    (property "LCSC" "C377773" (id 4) (at 53.975 83.185 0)
+    (property "LCSC" "C50254" (id 4) (at 53.975 83.185 0)
       (effects (font (size 1.27 1.27)) hide)
     )
@@
       (effects (font (size 1.27 1.27)) (justify left))
     )
-    (property "Footprint" "Capacitor_SMD:C_0805_2012Metric" (id 2) (at 77.47 151.13 0)
+    (property "Footprint" "Capacitor_SMD:C_1206_3216Metric" (id 2) (at 77.47 151.13 0)
       (effects (font (size 1.27 1.27)) hide)
     )
@@
       (effects (font (size 1.27 1.27)) hide)
     )
-    (property "LCSC" "C377773" (id 4) (at 77.47 151.13 0)
+    (property "LCSC" "C50254" (id 4) (at 77.47 151.13 0)
       (effects (font (size 1.27 1.27)) hide)
     )
@@
     )
     (path "/56a3fbd6-97b9-4085-a60a-8897c25832b9"
-      (reference "C5") (unit 1) (value "2u2") (footprint "Capacitor_SMD:C_0805_2012Metric")
+      (reference "C5") (unit 1) (value "2u2") (footprint "Capacitor_SMD:C_1206_3216Metric")
     )
     (path "/c2ff0469-2f48-48da-ad0d-212c22384264"
@@
     )
     (path "/6c555782-8a4f-4f13-890c-e84b5d734ffc"
-      (reference "C12") (unit 1) (value "2u2") (footprint "Capacitor_SMD:C_0805_2012Metric")
+      (reference "C12") (unit 1) (value "2u2") (footprint "Capacitor_SMD:C_1206_3216Metric")
     )
     (path "/95539020-f987-4434-820b-47502b6eeada"

Commit message: Doing calcs + removing caps that might introduce noise.
Parts:
- removed C17, C22: 22u, Capacitor_SMD:C_1210_3225Metric, symbol Device:C_Small
- removed D1: P6SMB20A, Diode_SMD:D_SMB, symbol Diode:SM6T15A
- removed FB1, FB2: 600Ω@100MHz, Resistor_SMD:R_0805_2012Metric, symbol Device:FerriteBead_Small
- added C10: C_Polarized_Small, Capacitor_SMD:CP_Elec_6.3x5.9, symbol Device:C_Polarized_Small
- added L1, L3: 10u, Inductor_SMD:L_0805_2012Metric, symbol Device:L_Small
- R12: renamed from R11; value 1k -> 6k8; LCSC C11702 -> C25917
- R13: value 1k -> 6k8; LCSC C11702 -> C25917
- renumbered C3 to C1, C6 to C11, C7 to C12, C8 to C14, C14 to C15, C15 to C16, C23 to C17, C16 to C19, C9 to C2, C19 to C20, C24 to C21, C20 to C22, C21 to C23, C25 to C24, C26 to C25, C1 to C3, C10 to C5, C5 to C6, C11 to C7, C12 to C8, C2 to C9, D2 to D1, D3 to D2, J6 to J3, J7 to J4, J8 to J5, J9 to J6, J3 to J7, J4 to J8, J5 to J9, L1 to L2, R12 to R10, R10 to R11, R5 to R3, R6 to R4, R7 to R5, R3 to R6, R4 to R7, U3 to U2, U2 to U3
Connections:
- net +10.5: now also L1.1
- net -10.5: now also L3.1
- net GND: now also C10.2
- net OUT_POS: now also L1.2
- net VCC: now also C10.1
- net at C15.2, C16.2, NT1.2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: now also L3.2

Commit message: Before restructuring max17579.
Parts:
- added R9: 27k 1%, Resistor_SMD:R_0402_1005Metric, symbol Device:R
- L2: footprint Inductor_SMD:L_Coilcraft_XAL60xx_6.36x6.56mm -> marcin_library:Wurth 74408063680
- R10: renamed from R9; value 1k78 1% -> 39k
- R8: value 19k1 1% -> 390k 1%
- renumbered R10 to R11, R11 to R12, R12 to R13, R13 to R14
Connections:
- net FB_NEG: now also R9.1; no longer R8.1
- new net: R8.1, R9.2
Other:
- moved on the sheet: R10, R8

Commit message: Fix footprints of MAX and MAXM.
Connections:
- net GND: now also L2.2; no longer L2.1
- net LX: now also L2.1; no longer L2.2
- net SOUT: now reaches C7.2, C8.2, NT1.1, R5.1, U2.13 (EP), U2.8 (SOUT)
Other:
- moved on the sheet: L2
Changed lines of the file:
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@@
+    (effects (font (size 1.27 1.27)) (justify left bottom))
+  )
+  (label "SOUT" (at 119.38 161.29 0)
     (effects (font (size 1.27 1.27)) (justify left bottom))
   )
@@
     (pin "2")
   )
-  (symbol (lib_id "Device:L_Small") (at 151.13 129.54 270) (mirror x) (unit 1)
+  (symbol (lib_id "Device:L_Small") (at 151.13 129.54 90) (unit 1)
     (in_bom yes) (on_board yes) (fields_autoplaced)
-    (property "Reference" "L2" (id 0) (at 151.13 124.46 90))
-    (property "Value" "47u" (id 1) (at 151.13 127 90))
+    (property "Reference" "L2" (id 0) (at 151.13 123.825 90))
+    (property "Value" "47u" (id 1) (at 151.13 126.365 90))
     (property "Footprint" "marcin_library:Wurth 74408063680" (id 2) (at 151.13 129.54 0)
       (effects (font (size 1.27 1.27)) hide)
